File: si-pcb.kicad_pcb (KiCad board)
At the start: 0 parts

Commit message: Create switches positions
Parts:
- added MX0: MX-NoLED, hitek725:Hitek725-1U, F.Cu at (12.7, 116.2)
- added MX1: MX-NoLED, hitek725:Hitek725-1U, F.Cu at (31.8, 116.2)
- added MX10: MX-NoLED, hitek725:Hitek725-1U, F.Cu at (203.2, 116.2)
- added MX11: MX-NoLED, hitek725:Hitek725-1U, F.Cu at (222.3, 116.2)
- added MX12: MX-NoLED, hitek725:Hitek725-1U, F.Cu at (241.3, 116.2)
- added MX13: MX-NoLED, hitek725:Hitek725-1U, F.Cu at (260.4, 116.2)
- added MX14-0: MX-NoLED, hitek725:Hitek725-1U, F.Cu at (279.4, 116.2)
- added MX14-1: MX-NoLED, hitek725:Hitek725-1U-reversed, F.Cu at (269.9, 116.2)
- added MX15-0: MX-NoLED, hitek725:Hitek725-1.5U, F.Cu at (17.5, 135.2)
- added MX15-1: MX-NoLED, hitek725:Hitek725-1.25U, F.Cu at (19.9, 135.2)
- added MX16: MX-NoLED, hitek725:Hitek725-1U, F.Cu at (41.3, 135.2)
- added MX17: MX-NoLED, hitek725:Hitek725-1U, F.Cu at (60.4, 135.2)
- added MX18: MX-NoLED, hitek725:Hitek725-1U, F.Cu at (79.4, 135.2)
- added MX19: MX-NoLED, hitek725:Hitek725-1U, F.Cu at (98.5, 135.2)
- added MX2: MX-NoLED, hitek725:Hitek725-1U, F.Cu at (50.8, 116.2)
- added MX20: MX-NoLED, hitek725:Hitek725-1U, F.Cu at (117.5, 135.2)
- added MX21: MX-NoLED, hitek725:Hitek725-1U, F.Cu at (136.6, 135.2)
- added MX22: MX-NoLED, hitek725:Hitek725-1U, F.Cu at (155.6, 135.2)
- added MX23: MX-NoLED, hitek725:Hitek725-1U, F.Cu at (174.7, 135.2)
- added MX24: MX-NoLED, hitek725:Hitek725-1U, F.Cu at (193.7, 135.2)
- added MX25: MX-NoLED, hitek725:Hitek725-1U, F.Cu at (212.8, 135.2)
- added MX26: MX-NoLED, hitek725:Hitek725-1U, F.Cu at (231.8, 135.2)
- added MX27: MX-NoLED, hitek725:Hitek725-1U, F.Cu at (250.9, 135.2)
- added MX28-0: MX-NoLED, hitek725:Hitek725-1.5U, F.Cu at (274.7, 135.2)
- added MX28-1: MX-NoLED, hitek725:Hitek725-1.25U, F.Cu at (272.3, 135.2)
- added MX29-0: MX-NoLED, hitek725:Hitek725-1.75U, F.Cu at (19.9, 154.3)
- added MX29-1: MX-NoLED, hitek725:Hitek725-1.5U, F.Cu at (17.5, 154.3)
- added MX3: MX-NoLED, hitek725:Hitek725-1U, F.Cu at (69.9, 116.2)
- added MX30: MX-NoLED, hitek725:Hitek725-1U, F.Cu at (46.1, 154.3)
- added MX31: MX-NoLED, hitek725:Hitek725-1U, F.Cu at (65.1, 154.3)
- added MX32: MX-NoLED, hitek725:Hitek725-1U, F.Cu at (84.2, 154.3)
- added MX33: MX-NoLED, hitek725:Hitek725-1U, F.Cu at (103.2, 154.3)
- added MX34: MX-NoLED, hitek725:Hitek725-1U, F.Cu at (122.3, 154.3)
- added MX35: MX-NoLED, hitek725:Hitek725-1U, F.Cu at (141.3, 154.3)
- added MX36: MX-NoLED, hitek725:Hitek725-1U, F.Cu at (160.4, 154.3)
- added MX37: MX-NoLED, hitek725:Hitek725-1U, F.Cu at (179.4, 154.3)
- added MX38: MX-NoLED, hitek725:Hitek725-1U, F.Cu at (198.5, 154.3)
- added MX39: MX-NoLED, hitek725:Hitek725-1U, F.Cu at (217.5, 154.3)
- added MX4: MX-NoLED, hitek725:Hitek725-1U, F.Cu at (88.9, 116.2)
- added MX40: MX-NoLED, hitek725:Hitek725-1U, F.Cu at (236.6, 154.3)
- added MX42-0: MX-NoLED, hitek725:Hitek725-2.25U, F.Cu at (267.5, 154.3)
- added MX42-1: MX-NoLED, hitek725:Hitek725-2U, F.Cu at (265.2, 154.3)
- added MX42-3: MX-NoLED-SI, hitek725:Hitek725-BigAssEnter-separated-pins, F.Cu at (269.9, 144.7)
- added MX42-4: MX-NoLED-SI, hitek725:Hitek725-BigAssEnter-separated-pins-reversed, F.Cu at (265.2, 144.7)
- added MX43-0: MX-NoLED, hitek725:Hitek725-2.25U, F.Cu at (24.7, 173.3)
- added MX43-1: MX-NoLED, hitek725:Hitek725-2U, F.Cu at (27.0, 173.3)
- added MX45: MX-NoLED, hitek725:Hitek725-1U, F.Cu at (55.6, 173.3)
- added MX46: MX-NoLED, hitek725:Hitek725-1U, F.Cu at (74.7, 173.3)
- added MX47: MX-NoLED, hitek725:Hitek725-1U, F.Cu at (93.7, 173.3)
- added MX48: MX-NoLED, hitek725:Hitek725-1U, F.Cu at (112.8, 173.3)
- added MX49: MX-NoLED, hitek725:Hitek725-1U, F.Cu at (131.8, 173.3)
- added MX5: MX-NoLED, hitek725:Hitek725-1U, F.Cu at (108.0, 116.2)
- added MX50: MX-NoLED, hitek725:Hitek725-1U, F.Cu at (150.9, 173.3)
- added MX51: MX-NoLED, hitek725:Hitek725-1U, F.Cu at (169.9, 173.3)
- added MX52: MX-NoLED, hitek725:Hitek725-1U, F.Cu at (189.0, 173.3)
- added MX53: MX-NoLED, hitek725:Hitek725-1U, F.Cu at (208.0, 173.3)
- added MX54: MX-NoLED, hitek725:Hitek725-1U, F.Cu at (227.1, 173.3)
- added MX55-0: MX-NoLED, hitek725:Hitek725-2.75U, F.Cu at (262.8, 173.3)
- added MX55-1: MX-NoLED, hitek725:Hitek725-1U-reversed, F.Cu at (258.0, 173.3)
- added MX56: MX-NoLED, hitek725:Hitek725-1.5U, F.Cu at (17.5, 192.4)
- added MX57: MX-NoLED, hitek725:Hitek725-1U, F.Cu at (41.3, 192.4)
- added MX58: MX-NoLED, hitek725:Hitek725-1.5U, F.Cu at (65.1, 192.4)
- added MX59: MX-NoLED, hitek725:Hitek725-7U, F.Cu at (146.1, 192.4)
- added MX6: MX-NoLED, hitek725:Hitek725-1U, F.Cu at (127.0, 116.2)
- added MX60: MX-NoLED, hitek725:Hitek725-1.5U, F.Cu at (227.1, 192.4)
- added MX61: MX-NoLED, hitek725:Hitek725-1U, F.Cu at (250.9, 192.4)
- added MX62: MX-NoLED, hitek725:Hitek725-1.5U, F.Cu at (274.7, 192.4)
- added MX7: MX-NoLED, hitek725:Hitek725-1U, F.Cu at (146.1, 116.2)
- added MX8: MX-NoLED, hitek725:Hitek725-1U, F.Cu at (165.1, 116.2)
- added MX9: MX-NoLED, hitek725:Hitek725-1U, F.Cu at (184.2, 116.2)
Other:
- board outline added: 284.7 x 94.2 mm
- copper layers 0 -> 2
