File: si-pcb.kicad_pcb (KiCad board)
At the start: 2 copper layers, 284.7 x 94.2 mm, 70 parts

Commit message: Edit BEA switch symbols
Parts:
- MX42-4: footprint hitek725:Hitek725-BigAssEnter-separated-pins-reversed -> hitek725:Hitek725-BigAssEnter-reversed
Changed lines of the file:
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@@
   (net 16 "Net-(D7-Pad2)")
   (net 17 "Col7")
-  (net 18 "Net-(MX8-Pad2)")
+  (net 18 "Net-(D8-Pad2)")
   (net 19 "Col8")
   (net 20 "Net-(D9-Pad2)")
@@
   (net 42 "Net-(D30-Pad2)")
   (net 43 "Net-(D31-Pad2)")
-  (net 44 "Net-(MX32-Pad2)")
+  (net 44 "Net-(D32-Pad2)")
   (net 45 "Net-(D33-Pad2)")
   (net 46 "Net-(D34-Pad2)")
@@
   (net 54 "Net-(D45-Pad2)")
   (net 55 "Net-(D46-Pad2)")
-  (net 56 "Net-(MX47-Pad2)")
+  (net 56 "Net-(D47-Pad2)")
   (net 57 "Net-(D48-Pad2)")
   (net 58 "Net-(D49-Pad2)")
@@
   (net 67 "Net-(D59-Pad2)")
   (net 68 "Net-(D60-Pad2)")
-  (net 69 "Net-(MX61-Pad2)")
+  (net 69 "Net-(D61-Pad2)")
   (net 70 "Net-(D62-Pad2)")
   (net 71 "Net-(D14-Pad2)")
@@
       (net 20 "Net-(D9-Pad2)") (pinfunction "ROW") (pintype "passive"))
   )
-  (footprint "hitek725:Hitek725-BigAssEnter-separated-pins-reversed" (layer "F.Cu")
+  (footprint "hitek725:Hitek725-BigAssEnter-reversed" (layer "F.Cu")
     (at 265.162386 144.731264)
     (property "Sheetfile" "si-pcb.kicad_sch")
@@
       (effects (font (size 1 1) (thickness 0.15)))
     )
-    (fp_line (start 19.05 19.05) (end -23.8125 19.05) (layer "Dwgs.User") (width 0.15))
-    (fp_line (start -9.525 0) (end -9.525 -19.05) (layer "Dwgs.User") (width 0.15))
     (fp_line (start -9.525 -19.05) (end 19.05 -19.05) (layer "Dwgs.User") (width 0.15))
-    (fp_line (start -23.8125 0) (end -23.8125 19.05) (layer "Dwgs.User") (width 0.15))
     (fp_line (start 19.05 -19.05) (end 19.05 19.05) (layer "Dwgs.User") (width 0.15))
     (fp_line (start -9.525 0) (end -23.8125 0) (layer "Dwgs.User") (width 0.15))
+    (fp_line (start 19.05 19.05) (end -23.8125 19.05) (layer "Dwgs.User") (width 0.15))
+    (fp_line (start -23.8125 0) (end -23.8125 19.05) (layer "Dwgs.User") (width 0.15))
+    (fp_line (start -9.525 0) (end -9.525 -19.05) (layer "Dwgs.User") (width 0.15))
     (pad "1" thru_hole circle (at 5.08 -3.3) (size 3.18 3.18) (drill 1.4) (layers *.Cu *.Mask)
       (net 29 "Col13") (pinfunction "COL") (pintype "passive"))
+    (pad "1" thru_hole circle (at -0.64 -3.3) (size 3.18 3.18) (drill 1.4) (layers *.Cu *.Mask)
+      (net 29 "Col13") (pinfunction "COL") (pintype "passive"))
+    (pad "2" thru_hole circle (at -0.64 3.3) (size 3.18 3.18) (drill 1.4) (layers *.Cu *.Mask)
+      (net 75 "Net-(D42-Pad2)") (pinfunction "ROW") (pintype "passive"))
     (pad "2" thru_hole circle (at 5.08 3.3) (size 3.18 3.18) (drill 1.4) (layers *.Cu *.Mask)
       (net 75 "Net-(D42-Pad2)") (pinfunction "ROW") (pintype "passive"))
-    (pad "2" thru_hole circle (at -0.64 3.3) (size 3.18 3.18) (drill 1.4) (layers *.Cu *.Mask)
-      (net 75 "Net-(D42-Pad2)") (pinfunction "ROW") (pintype "passive"))
-    (pad "3" thru_hole circle (at -0.64 -3.3) (size 3.18 3.18) (drill 1.4) (layers *.Cu *.Mask))
   )
   (footprint "hitek725:Hitek725-1U" (layer "F.Cu")
@@
       (net 9 "Col3") (pinfunction "COL") (pintype "passive"))
     (pad "2" thru_hole circle (at 3.3 5.08) (size 3.18 3.18) (drill 1.4) (layers *.Cu *.Mask)
-      (net 44 "Net-(MX32-Pad2)") (pinfunction "ROW") (pintype "passive"))
-    (pad "2" thru_hole circle (at 3.3 -0.64) (size 3.18 3.18) (drill 1.4) (layers *.Cu *.Mask)
-      (net 44 "Net-(MX32-Pad2)") (pinfunction "ROW") (pintype "passive"))
+      (net 44 "Net-(D32-Pad2)") (pinfunction "ROW") (pintype "passive"))
+    (pad "2" thru_hole circle (at 3.3 -0.64) (size 3.18 3.18) (drill 1.4) (layers *.Cu *.Mask)
+      (net 44 "Net-(D32-Pad2)") (pinfunction "ROW") (pintype "passive"))
   )
   (footprint "hitek725:Hitek725-1U" (layer "F.Cu")
@@
       (net 11 "Col4") (pinfunction "COL") (pintype "passive"))
     (pad "2" thru_hole circle (at 3.3 5.08) (size 3.18 3.18) (drill 1.4) (layers *.Cu *.Mask)
-      (net 56 "Net-(MX47-Pad2)") (pinfunction "ROW") (pintype "passive"))
-    (pad "2" thru_hole circle (at 3.3 -0.64) (size 3.18 3.18) (drill 1.4) (layers *.Cu *.Mask)
-      (net 56 "Net-(MX47-Pad2)") (pinfunction "ROW") (pintype "passive"))
+      (net 56 "Net-(D47-Pad2)") (pinfunction "ROW") (pintype "passive"))
+    (pad "2" thru_hole circle (at 3.3 -0.64) (size 3.18 3.18) (drill 1.4) (layers *.Cu *.Mask)
+      (net 56 "Net-(D47-Pad2)") (pinfunction "ROW") (pintype "passive"))
   )
   (footprint "hitek725:Hitek725-1U" (layer "F.Cu")
@@
       (net 27 "Col12") (pinfunction "COL") (pintype "passive"))
     (pad "2" thru_hole circle (at 3.3 -0.64) (size 3.18 3.18) (drill 1.4) (layers *.Cu *.Mask)
-      (net 69 "Net-(MX61-Pad2)") (pinfunction "ROW") (pintype "passive"))
-    (pad "2" thru_hole circle (at 3.3 5.08) (size 3.18 3.18) (drill 1.4) (layers *.Cu *.Mask)
-      (net 69 "Net-(MX61-Pad2)") (pinfunction "ROW") (pintype "passive"))
+      (net 69 "Net-(D61-Pad2)") (pinfunction "ROW") (pintype "passive"))
+    (pad "2" thru_hole circle (at 3.3 5.08) (size 3.18 3.18) (drill 1.4) (layers *.Cu *.Mask)
+      (net 69 "Net-(D61-Pad2)") (pinfunction "ROW") (pintype "passive"))
   )
   (footprint "hitek725:Hitek725-1U" (layer "F.Cu")
@@
       (net 19 "Col8") (pinfunction "COL") (pintype "passive"))
     (pad "2" thru_hole circle (at 3.3 -0.64) (size 3.18 3.18) (drill 1.4) (layers *.Cu *.Mask)
-      (net 18 "Net-(MX8-Pad2)") (pinfunction "ROW") (pintype "passive"))
-    (pad "2" thru_hole circle (at 3.3 5.08) (size 3.18 3.18) (drill 1.4) (layers *.Cu *.Mask)
-      (net 18 "Net-(MX8-Pad2)") (pinfunction "ROW") (pintype "passive"))
-  )
-  (footprint "hitek725:Hitek725-1U" (layer "F.Cu")
+      (net 18 "Net-(D8-Pad2)") (pinfunction "ROW") (pintype "passive"))
+    (pad "2" thru_hole circle (at 3.3 5.08) (size 3.18 3.18) (drill 1.4) (layers *.Cu *.Mask)
+      (net 18 "Net-(D8-Pad2)") (pinfunction "ROW") (pintype "passive"))
+  )
+  (footprint "hitek725:Hitek725-1U" (layer "F.Cu")
