File: si-pcb.kicad_sch (KiCad schematic)
At the start: 0 parts

Commit message: Create switches positions
Parts:
- added D0, D1, D10, D11, D12, D13, D14, D15, D16, D17, D18, D19, D2, D20, D21, D22, D23, D24, D25, D26, D27, D28, D29, D3, D30, D31, D32, D33, D34, D35, D36, D37, D38, D39, D4, D40, D42, D43, D45, D46, D47, D48, D49, D5, D50, D51, D52, D53, D54, D55, D56, D57, D58, D59, D6, D60, D61, D62, D7, D8, D9: D_Small, symbol Device:D_Small
- added MX0, MX1, MX10, MX11, MX12, MX13, MX14-0, MX16, MX17, MX18, MX19, MX2, MX20, MX21, MX22, MX23, MX24, MX25, MX26, MX27, MX3, MX30, MX31, MX32, MX33, MX34, MX35, MX36, MX37, MX38, MX39, MX4, MX40, MX45, MX46, MX47, MX48, MX49, MX5, MX50, MX51, MX52, MX53, MX54, MX57, MX6, MX61, MX7, MX8, MX9: MX-NoLED, hitek725:Hitek725-1U, symbol MX_Alps_Hybrid:MX-NoLED
- added MX14-1, MX55-1: MX-NoLED, hitek725:Hitek725-1U-reversed, symbol MX_Alps_Hybrid:MX-NoLED
- added MX15-0, MX28-0, MX29-1, MX56, MX58, MX60, MX62: MX-NoLED, hitek725:Hitek725-1.5U, symbol MX_Alps_Hybrid:MX-NoLED
- added MX15-1, MX28-1: MX-NoLED, hitek725:Hitek725-1.25U, symbol MX_Alps_Hybrid:MX-NoLED
- added MX29-0: MX-NoLED, hitek725:Hitek725-1.75U, symbol MX_Alps_Hybrid:MX-NoLED
- added MX42-0, MX43-0: MX-NoLED, hitek725:Hitek725-2.25U, symbol MX_Alps_Hybrid:MX-NoLED
- added MX42-1, MX43-1: MX-NoLED, hitek725:Hitek725-2U, symbol MX_Alps_Hybrid:MX-NoLED
- added MX42-3: MX-NoLED-SI, hitek725:Hitek725-BigAssEnter-separated-pins, symbol MX_Alps_Hybrid:MX-NoLED-SI
- added MX42-4: MX-NoLED-SI, hitek725:Hitek725-BigAssEnter-separated-pins-reversed, symbol MX_Alps_Hybrid:MX-NoLED-SI
- added MX55-0: MX-NoLED, hitek725:Hitek725-2.75U, symbol MX_Alps_Hybrid:MX-NoLED
- added MX59: MX-NoLED, hitek725:Hitek725-7U, symbol MX_Alps_Hybrid:MX-NoLED
Connections:
- new net: D56.2 (A), MX56.2 (ROW)
- new net: D45.2 (A), MX45.2 (ROW)
- new net: D9.2 (A), MX9.2 (ROW)
- new net: D29.2 (A), MX29-0.2 (ROW), MX29-1.2 (ROW)
- new net: D47.2 (A), MX47.2 (ROW)
- new net: D22.2 (A), MX22.2 (ROW)
- new net: D31.2 (A), MX31.2 (ROW)
- new net: D58.2 (A), MX58.2 (ROW)
- new net: D62.2 (A), MX62.2 (ROW)
- new net: D48.2 (A), MX48.2 (ROW)
- new net: D59.2 (A), MX59.2 (ROW)
- new net: D24.2 (A), MX24.2 (ROW)
- new net: D39.2 (A), MX39.2 (ROW)
- new net: D1.2 (A), MX1.2 (ROW)
- new net: D43.2 (A), MX43-0.2 (ROW), MX43-1.2 (ROW)
- new net: D37.2 (A), MX37.2 (ROW)
- new net: D18.2 (A), MX18.2 (ROW)
- new net: D5.2 (A), MX5.2 (ROW)
- new net: D52.2 (A), MX52.2 (ROW)
- new net: D33.2 (A), MX33.2 (ROW)
- new net: D61.2 (A), MX61.2 (ROW)
- new net: D27.2 (A), MX27.2 (ROW)
- new net: D40.2 (A), MX40.2 (ROW)
- new net: D35.2 (A), MX35.2 (ROW)
- new net: D17.2 (A), MX17.2 (ROW)
- new net: D38.2 (A), MX38.2 (ROW)
- new net: D12.2 (A), MX12.2 (ROW)
- new net: D49.2 (A), MX49.2 (ROW)
- new net: D20.2 (A), MX20.2 (ROW)
- new net: D8.2 (A), MX8.2 (ROW)
- new net: D50.2 (A), MX50.2 (ROW)
- new net: D0.2 (A), MX0.2 (ROW)
- new net: D13.2 (A), MX13.2 (ROW)
- new net: D28.2 (A), MX28-0.2 (ROW), MX28-1.2 (ROW)
- new net: D23.2 (A), MX23.2 (ROW)
- new net: D55.2 (A), MX55-0.2 (ROW), MX55-1.2 (ROW)
- new net: D51.2 (A), MX51.2 (ROW)
- new net: D25.2 (A), MX25.2 (ROW)
- new net: D54.2 (A), MX54.2 (ROW)
- new net: D21.2 (A), MX21.2 (ROW)
- new net: D34.2 (A), MX34.2 (ROW)
- new net: D46.2 (A), MX46.2 (ROW)
- new net: D15.2 (A), MX15-0.2 (ROW), MX15-1.2 (ROW)
- new net: D42.2 (A), MX42-0.2 (ROW), MX42-1.2 (ROW), MX42-3.2 (ROW), MX42-4.2 (ROW)
- new net: D32.2 (A), MX32.2 (ROW)
- new net: D11.2 (A), MX11.2 (ROW)
- new net: D60.2 (A), MX60.2 (ROW)
- new net: D36.2 (A), MX36.2 (ROW)
- new net: D7.2 (A), MX7.2 (ROW)
- new net: D53.2 (A), MX53.2 (ROW)
- new net: D10.2 (A), MX10.2 (ROW)
- new net: D14.2 (A), MX14-0.2 (ROW), MX14-1.2 (ROW)
- new net: D57.2 (A), MX57.2 (ROW)
- new net: D30.2 (A), MX30.2 (ROW)
- new net: D16.2 (A), MX16.2 (ROW)
- new net: D19.2 (A), MX19.2 (ROW)
- new net: D2.2 (A), MX2.2 (ROW)
- new net: D6.2 (A), MX6.2 (ROW)
- new net: D26.2 (A), MX26.2 (ROW)
- new net: D3.2 (A), MX3.2 (ROW)
- new net: D4.2 (A), MX4.2 (ROW)
- new net Col0: MX0.1 (COL), MX15-0.1 (COL), MX15-1.1 (COL), MX29-0.1 (COL), MX29-1.1 (COL), MX43-0.1 (COL), MX43-1.1 (COL), MX56.1 (COL)
- new net Col1: MX1.1 (COL), MX16.1 (COL), MX30.1 (COL), MX57.1 (COL)
- new net Col10: MX10.1 (COL), MX25.1 (COL), MX39.1 (COL), MX53.1 (COL)
- new net Col11: MX11.1 (COL), MX26.1 (COL), MX40.1 (COL), MX54.1 (COL), MX60.1 (COL)
- new net Col12: MX12.1 (COL), MX27.1 (COL), MX55-0.1 (COL), MX55-1.1 (COL), MX61.1 (COL)
- new net Col13: MX13.1 (COL), MX28-0.1 (COL), MX28-1.1 (COL), MX42-0.1 (COL), MX42-1.1 (COL), MX42-3.1 (COL), MX42-4.1 (COL), MX62.1 (COL)
- new net Col14: MX14-0.1 (COL), MX14-1.1 (COL)
- new net Col2: MX17.1 (COL), MX2.1 (COL), MX31.1 (COL), MX45.1 (COL), MX58.1 (COL)
- new net Col3: MX18.1 (COL), MX3.1 (COL), MX32.1 (COL), MX46.1 (COL)
- new net Col4: MX19.1 (COL), MX33.1 (COL), MX4.1 (COL), MX47.1 (COL)
- new net Col5: MX20.1 (COL), MX34.1 (COL), MX48.1 (COL), MX5.1 (COL)
- new net Col6: MX21.1 (COL), MX35.1 (COL), MX49.1 (COL), MX59.1 (COL), MX6.1 (COL)
- new net Col7: MX22.1 (COL), MX36.1 (COL), MX50.1 (COL), MX7.1 (COL)
- new net Col8: MX23.1 (COL), MX37.1 (COL), MX51.1 (COL), MX8.1 (COL)
- new net Col9: MX24.1 (COL), MX38.1 (COL), MX52.1 (COL), MX9.1 (COL)
- new net Row0: D0.1 (K), D1.1 (K), D10.1 (K), D11.1 (K), D12.1 (K), D13.1 (K), D14.1 (K), D2.1 (K), D3.1 (K), D4.1 (K), D5.1 (K), D6.1 (K), D7.1 (K), D8.1 (K), D9.1 (K)
- new net Row1: D15.1 (K), D16.1 (K), D17.1 (K), D18.1 (K), D19.1 (K), D20.1 (K), D21.1 (K), D22.1 (K), D23.1 (K), D24.1 (K), D25.1 (K), D26.1 (K), D27.1 (K), D28.1 (K)
- new net Row2: D29.1 (K), D30.1 (K), D31.1 (K), D32.1 (K), D33.1 (K), D34.1 (K), D35.1 (K), D36.1 (K), D37.1 (K), D38.1 (K), D39.1 (K), D40.1 (K), D42.1 (K)
- new net Row3: D43.1 (K), D45.1 (K), D46.1 (K), D47.1 (K), D48.1 (K), D49.1 (K), D50.1 (K), D51.1 (K), D52.1 (K), D53.1 (K), D54.1 (K), D55.1 (K), D56.1 (K), D57.1 (K), D58.1 (K), D59.1 (K), D60.1 (K), D61.1 (K), D62.1 (K)
